File: RBF PCB/RBF PCB.kicad_pcb (KiCad board)
At the start: 2 copper layers, 40 x 70 mm, 10 parts, among them J1 DF11-12DP, J2 DF11-12DP, J5 DF11-12DP, J6 DF11-12DP, J9 B2B-XH-A

Commit message: manufacturing files
Parts:
- moved J5 76.9 mm to (167.3, 114.4)
- moved J6 76.9 mm to (167.3, 93.3)
- moved H1 76.9 mm to (139.3, 75.3)
- moved H2 76.9 mm to (139.3, 135.3)
- moved H3 76.9 mm to (168.3, 75.3)
- moved H4 76.9 mm to (168.3, 135.3)
- moved J1 76.9 mm to (138.3, 114.4)
- moved J2 76.9 mm to (138.3, 93.3)
- moved J9 76.9 mm to (168.3, 123.9)
- moved SW1 76.9 mm to (147.5, 91.0)
Routing:
- net NC: track 67.4 -> 78.9 mm
Other:
- board text added: "GND"
- board text added: "NC"
- board text added: "left VBat+ Right Vbat-"
Changed lines of the file:
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@@
 			(outputformat 1)
 			(mirror no)
-			(drillshape 1)
+			(drillshape 0)
 			(scaleselection 1)
 			(outputdirectory "")
@@
 	(footprint "MountingHole:MountingHole_2.7mm_M2.5_Pad_Via"
 		(layer "F.Cu")
-		(at 100 100)
+		(at 168.2875 135.3125)
 		(descr "Mounting Hole 2.7mm, M2.5, generated by kicad-footprint-generator mountinghole.py")
 		(tags "mountinghole M2.5")
@@
 	(footprint "DF-11:JST_B2B-XH-A"
 		(layer "F.Cu")
-		(at 100 88.58 90)
+		(at 168.2875 123.8925 90)
 		(property "Reference" "J9"
 			(at -0.54 -1.4 90)
@@
 	(footprint "Connector_Hirose:Hirose_DF11-12DP-2DSA_2x06_P2.00mm_Vertical"
 		(layer "F.Cu")
-		(at 70 79.06 90)
+		(at 138.2875 114.3725 90)
 		(descr "Hirose DF11 through hole, DF11-12DP-2DSA, 6 Pins per row (https://www.hirose.com/product/document?clcode=&productname=&series=DF11&documenttype=Catalog&lang=en&documentid=D31688_en)")
 		(tags "connector Hirose DF11 vertical")
@@
 	(footprint "Connector_Hirose:Hirose_DF11-12DP-2DSA_2x06_P2.00mm_Vertical"
 		(layer "F.Cu")
-		(at 99.05 79.06 90)
+		(at 167.3375 114.3725 90)
 		(descr "Hirose DF11 through hole, DF11-12DP-2DSA, 6 Pins per row (https://www.hirose.com/product/document?clcode=&productname=&series=DF11&documenttype=Catalog&lang=en&documentid=D31688_en)")
 		(tags "connector Hirose DF11 vertical")
@@
 	(footprint "Connector_Hirose:Hirose_DF11-12DP-2DSA_2x06_P2.00mm_Vertical"
 		(layer "F.Cu")
-		(at 70 57.99 90)
+		(at 138.2875 93.3025 90)
 		(descr "Hirose DF11 through hole, DF11-12DP-2DSA, 6 Pins per row (https://www.hirose.com/product/document?clcode=&productname=&series=DF11&documenttype=Catalog&lang=en&documentid=D31688_en)")
 		(tags "connector Hirose DF11 vertical")
@@
 	(footprint "FOOT print libary:RBF Switch foot print"
 		(layer "F.Cu")
-		(at 79.25 55.7 -90)
+		(at 147.5375 91.0125 -90)
 		(property "Reference" "SW1"
 			(at 1.5 -2 270)
@@
 	(footprint "MountingHole:MountingHole_2.7mm_M2.5_Pad_Via"
 		(layer "F.Cu")
-		(at 71 100)
+		(at 139.2875 135.3125)
 		(descr "Mounting Hole 2.7mm, M2.5, generated by kicad-footprint-generator mountinghole.py")
 		(tags "mountinghole M2.5")
@@
 	(footprint "Connector_Hirose:Hirose_DF11-12DP-2DSA_2x06_P2.00mm_Vertical"
 		(layer "F.Cu")
-		(at 99.05 57.99 90)
+		(at 167.3375 93.3025 90)
 		(descr "Hirose DF11 through hole, DF11-12DP-2DSA, 6 Pins per row (https://www.hirose.com/product/document?clcode=&productname=&series=DF11&documenttype=Catalog&lang=en&documentid=D31688_en)")
 		(tags "connector Hirose DF11 vertical")
@@
 	(footprint "MountingHole:MountingHole_2.7mm_M2.5_Pad_Via"
 		(layer "F.Cu")
-		(at 100 40)
+		(at 168.2875 75.3125)
 		(descr "Mounting Hole 2.7mm, M2.5, generated by kicad-footprint-generator mountinghole.py")
 		(tags "mountinghole M2.5")
@@
 	(footprint "MountingHole:MountingHole_2.7mm_M2.5_Pad_Via"
 		(layer "F.Cu")
-		(at 71 40)
+		(at 139.2875 75.3125)
 		(descr "Mounting Hole 2.7mm, M2.5, generated by kicad-footprint-generator mountinghole.py")
 		(tags "mountinghole M2.5")
@@
 	)
 	(gr_arc
-		(start 66 40)
-		(mid 67.464466 36.464466)
-		(end 71 35)
+		(start 134.2875 75.3125)
+		(mid 135.751966 71.776966)
+		(end 139.2875 70.3125)
 		(stroke
 			(width 0.2)
@@
 	)
 	(gr_line
-		(start 66 100)
-		(end 66 40)
+		(start 134.2875 135.3125)
+		(end 134.2875 75.3125)
 		(stroke
 			(width 0.2)
@@
 	)
 	(gr_line
-		(start 71 35)
-		(end 101 35)
+		(start 139.2875 70.3125)
+		(end 169.2875 70.3125)
 		(stroke
 			(width 0.2)
@@
 	)
 	(gr_arc
-		(start 71 105)
-		(mid 67.464466 103.535534)
-		(end 66 100)
+		(start 139.2875 140.3125)
+		(mid 135.751966 138.848034)
+		(end 134.2875 135.3125)
 		(stroke
 			(width 0.2)
@@
 	)
 	(gr_arc
-		(start 101 35)
-		(mid 104.535534 36.464466)
-		(end 106 40)
+		(start 169.2875 70.3125)
+		(mid 172.823034 71.776966)
+		(end 174.2875 75.3125)
 		(stroke
 			(width 0.2)
@@
 	)
 	(gr_line
-		(start 101 105)
-		(end 71 105)
+		(start 169.2875 140.3125)
+		(end 139.2875 140.3125)
 		(stroke
 			(width 0.2)
@@
 	)
 	(gr_line
-		(start 106 40)
-		(end 106 100)
+		(start 174.2875 75.3125)
+		(end 174.2875 135.3125)
 		(stroke
 			(width 0.2)
@@
 	)
 	(gr_arc
-		(start 106 100)
-		(mid 104.535534 103.535534)
-		(end 101 105)
+		(start 174.2875 135.3125)
+		(mid 172.823034 138.848034)
+		(end 169.2875 140.3125)
 		(stroke
 			(width 0.2)
@@
 		(layer "Edge.Cuts")
 	)
+	(gr_text "left VBat+	\nRight Vbat-\n"
+		(at 136.3775 121.4625 0)
+		(layer "F.SilkS")
+		(effects
+			(font
+				(size 1 1)
+				(thickness 0.15)
+			)
+			(justify left bottom)
+		)
+	)
 	(gr_text "pack in \n"
-		(at 67.97 66.37 90)
+		(at 136.2575 101.6825 90)
 		(layer "F.SilkS")
 		(effects
@@
 	)
 	(gr_text "Thermal board\n\n\n"
-		(at 99.21 94.24 90)
+		(at 167.4975 129.5525 90)
+		(layer "F.SilkS")
+		(effects
+			(font
+				(size 1 1)
+				(thickness 0.15)
+			)
+			(justify left bottom)
+		)
+	)
+	(gr_text "NC\n"
+		(at 171.1625 123.337989 90)
+		(layer "F.SilkS")
+		(effects
+			(font
+				(size 1 1)
+				(thickness 0.15)
+			)
+			(justify left bottom)
+		)
+	)
+	(gr_text "GND\n"
+		(at 171.1625 127.5925 90)
 		(layer "F.SilkS")
 		(effects
@@
 	)
 	(gr_text "pack out\n \n"
-		(at 102.46 60.19 270)
+		(at 170.7475 95.5025 270)
 		(layer "F.SilkS")
 		(effects
@@
 	)
 	(segment
-		(start 100.525 87.33)
-		(end 100.525 80.535)
+		(start 167.3375 110.3725)
+		(end 167.3375 112.3725)
 		(width 0.7)
 		(layer "F.Cu")
@@
 	)
 	(segment
-		(start 100.525 80.535)
-		(end 99.05 79.06)
+		(start 167.3375 108.3725)
+		(end 167.3375 110.3725)
 		(width 0.7)
 		(layer "F.Cu")
@@
 	)
 	(segment
-		(start 99.05 73.06)
-		(end 99.05 71.06)
+		(start 167.3375 112.3725)
+		(end 167.3375 114.3725)
 		(width 0.7)
 		(layer "F.Cu")
@@
 	)
 	(segment
-		(start 99.05 79.06)
-		(end 99.05 77.06)
+		(start 165.9625 104.9975)
+		(end 167.3375 106.3725)
 		(width 0.7)
 		(layer "F.Cu")
@@
 	)
 	(segment
-		(start 99.05 71.06)
-		(end 97.67 69.68)
+		(start 167.3375 93.3025)
+		(end 165.9625 94.6775)
 		(width 0.7)
 		(layer "F.Cu")
@@
 	)
 	(segment
-		(start 99.05 55.99)
-		(end 99.05 53.99)
+		(start 167.3375 85.3025)
+		(end 167.3375 87.3025)
 		(width 0.7)
 		(layer "F.Cu")
@@
 	)
 	(segment
-		(start 99.05 57.99)
-		(end 99.05 55.99)
+		(start 154.3275 108.1575)
+		(end 168.8125 122.6425)
 		(width 0.7)
 		(layer "F.Cu")
@@
 	)
 	(segment
-		(start 99.05 51.99)
-		(end 99.05 49.99)
+		(start 154.3275 100.3525)
+		(end 154.3275 108.1575)
 		(width 0.7)
 		(layer "F.Cu")
@@
 	)
 	(segment
-		(start 86.04 72.845)
-		(end 100.525 87.33)
+		(start 167.3375 91.3025)
+		(end 167.3375 93.3025)
 		(width 0.7)
 		(layer "F.Cu")
@@
 	)
 	(segment
-		(start 86.04 65.04)
-		(end 86.04 72.845)
+		(start 154.3275 98.3125)
+		(end 167.3375 85.3025)
 		(width 0.7)
 		(layer "F.Cu")
@@
 	)
 	(segment
-		(start 97.67 59.37)
-		(end 99.05 57.99)
+		(start 165.9625 94.6775)
+		(end 165.9625 104.9975)
 		(width 0.7)
 		(layer "F.Cu")
@@
 	)
 	(segment
-		(start 97.67 69.68)
-		(end 97.67 59.37)
+		(start 167.3375 106.3725)
+		(end 167.3375 108.3725)
 		(width 0.7)
 		(layer "F.Cu")
@@
 	)
 	(segment
-		(start 99.05 77.06)
-		(end 99.05 75.06)
+		(start 167.3375 87.3025)
+		(end 167.3375 89.3025)
 		(width 0.7)
 		(layer "F.Cu")
@@
 	)
 	(segment
-		(start 99.05 53.99)
-		(end 99.05 51.99)
+		(start 154.3275 100.3525)
+		(end 154.3275 98.3125)
 		(width 0.7)
 		(layer "F.Cu")
@@
 	)
 	(segment
-		(start 99.05 75.06)
-		(end 99.05 73.06)
+		(start 167.3375 89.3025)
+		(end 167.3375 91.3025)
 		(width 0.7)
 		(layer "F.Cu")
@@
 	)
 	(segment
-		(start 72 49.99)
-		(end 72.33 50.32)
+		(start 140.2875 85.3025)
+		(end 140.6175 85.6325)
 		(width 0.2)
 		(layer "B.Cu")
@@
 		(polygon
 			(pts
-				(xy 64.63 33.64) (xy 107.01 34) (xy 107.17 105.71) (xy 64.32 105.8)
+				(xy 132.9175 68.9525) (xy 175.2975 69.3125) (xy 175.4575 141.0225) (xy 132.6075 141.1125)
 			)
 		)
@@
 		(polygon
 			(pts
-				(xy 64.63 33.64) (xy 107.01 34) (xy 107.17 105.71) (xy 64.32 105.8)
+				(xy 132.9175 68.9525) (xy 175.2975 69.3125) (xy 175.4575 141.0225) (xy 132.6075 141.1125)
 			)
 		)
